File: KiCad/nex.kicad_pcb (KiCad board)
At the start: 2 copper layers, 35 x 39 mm, 62 parts, among them J1 BATT_JST, J2 USB_C_Receptacle_USB2.0_14P, J3 MOTOR_A, J4 MOTOR_B, Q1 FS8205A, SW1 SW_SPST, SW2 RESET, SW3 BOOT, SW4 SOC, U1 DW01A, U2 TP4056, U3 AP2112K-3.3TRG1, U4 ESP32-C3-WROOM-02-N4, U5 DRV8833PWPR, U6 MT3608, U7 74AHCT1G125W5-7, U8 STC3100IST

Commit message: readme
Parts:
- removed dialgorithm (x2): dialgorithm, dialgorithm:dialgorithm

Commit message: 4 layer update
Parts:
- U3: moved to B.Cu
- moved R8 29.4 mm to (113.5, 87.0), turned to 180 degrees
- moved R11 28.9 mm to (108.5, 86.0), turned to 0 degrees
- moved R10 25.1 mm to (110.0, 72.5)
- moved R12 25.1 mm to (107.5, 72.5)
- moved R7 25.1 mm to (112.5, 72.5)
- moved SW2 23.5 mm to (113.0, 82.5)
- moved R13 23.2 mm to (114.5, 83.0)
- moved R4 23.2 mm to (112.0, 83.0)
- moved R9 22.2 mm to (117.0, 83.0)
- moved D1 21.7 mm to (135.0, 80.5), turned to 180 degrees
- moved Q1 20.5 mm to (135.0, 76.5), turned to 180 degrees
- moved U5 19.7 mm to (109.9, 77.8), turned to 0 degrees
- moved U6 16.0 mm to (108.5, 92.5)
- moved C1 14.8 mm to (115.0, 78.0)
- moved R18 14.8 mm to (117.5, 78.0)
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- renumbered RCG to RCG1
Routing:
- net (no net): track 4.00 -> 0.00 mm
